Commit message: Update testbot.urdf

File: testbot_description/urdf/testbot.urdf (robot description, URDF)
Before this commit: robot test_robot, 5 links, 4 joints
Joints:
- joint joint1: origin xyz=0 0 0.25 rpy=0 0 0 -> xyz=0 0 0.5 rpy=0 0 0
- joint joint2: origin xyz=0 0 0.75 rpy=0 0 0 -> xyz=0 0 0.5 rpy=0 0 0
